File: USB-C.kicad_sch (KiCad schematic)
At the start: 7 parts, among them J301 USB_C_Receptacle_USB2.0, J302 JST - 1.00mm 4 Pin, U301 USBLC6-2SC6

Commit message: push de modification
Parts:
- removed J301: USB_C_Receptacle_USB2.0, Connector_USB:USB_C_Receptacle_GCT_USB4085, symbol Connector:USB_C_Receptacle_USB2.0
- added J2: USB_C_2-0, Connector_USB:USB_C_Receptacle_G-Switch_GT-USB-7010ASV, symbol Connector:USB_C_Receptacle_USB2.0
- F2: renamed from F301; footprint Fuse:Fuse_0402_1005Metric -> Fuse:Fuse_0805_2012Metric
- FB1: renamed from FB301; value 100 Ohm @ 100 MHz -> 600 Ohm @ 100 MHz; footprint Inductor_SMD:L_0402_1005Metric -> Inductor_SMD:L_0805_2012Metric
- R7: renamed from R301; footprint Resistor_SMD:R_0402_1005Metric -> Resistor_SMD:R_0603_1608Metric
- R8: renamed from R302; footprint Resistor_SMD:R_0402_1005Metric -> Resistor_SMD:R_0603_1608Metric
- renumbered J302 to J3, U301 to U5
Connections:
- net D1+: now also J2.A6 (D+), J2.B6 (D+)
- net D1-: now also J2.A7 (D-), J2.B7 (D-)
- net GND: now also J2.A1 (GND), J2.A12 (GND), J2.B1 (GND), J2.B12 (GND), J2.S1 (SHIELD)
- net VBUS: now also J3.1 (Pin_1), J2.A4 (VBUS), J2.A9 (VBUS), J2.B4 (VBUS), J2.B9 (VBUS)
- net at R7.2: now also J2.B5 (CC2)
- net at R8.2: now also J2.A5 (CC1)
- net VFused_ renamed V_Fused
- net V_Fused: no longer J3.1 (Pin_1)
- no-connect marks 3 -> 2
Other:
- note added: "PROTECTION"
- moved on the sheet: F2, FB1, J3, U5
